File: Hardware/SparkFun_HSTX_PTH_Breakout.kicad_sch (KiCad schematic)
At the start: 8 parts, among them J1 Conn_01x22_FPC_0.5mm_RA, J2 Conn_01x17

Commit message: Add dates
Parts:
- J1: PROD_ID (none) -> CONN-25634
Changed lines of the file:
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@@
 	(title_block
 		(title "SparkFun HSTX PTH Breakout")
+		(date "2025-03-03")
 		(rev "v10")
 		(company "SparkFun Electronics")
@@
 			)
 		)
-		(property "PROD_ID" ""
+		(property "PROD_ID" "CONN-25634"
 			(at 114.046 63.754 0)
 			(effects
